File: DX32MINI.kicad_sch (KiCad schematic)
At the start: 15 parts, among them J1 USB_B_Micro, J2 MicroSD Card, J3 GPIO - Left, J4 GPIO - Right, J5 Reset and Boot pins, SW1 reset, SW2 boot, U1 ESP32-S3-WROOM-1, U2 AMS1117-3.3

Commit message: Add files via upload
Parts:
- removed J5: Reset and Boot pins, Connector_PinHeader_2.54mm:PinHeader_1x02_P2.54mm_Vertical, symbol Connector_Generic:Conn_01x02
- added TP1, TP2: RESET, TestPoint:TestPoint_Pad_1.5x1.5mm, symbol Connector:TestPoint
- renumbered J3 to J2, J4 to J3, J2 to J4, SW2 to SW1, SW1 to SW2
Connections:
- net BOOT: now also TP2.1
- net RESET: now also TP1.1
Other:
- title: DX32A DELUXE Mini  -> DX32A DELUXE
